Commit message: imu urdf update

File: src/bfmc_car_description/urdf/bfmc_car_description.urdf.xacro (robot description, xacro)
@@ -465,4 +465,11 @@
     <child link="gps_tag_link"/>
     <origin xyz="0.135 0 0.102" rpy="0 0 0"/>
+  </joint>
+  <!-- Rear IMU (BNO055) — position from SolidWorks assembly export -->
+  <link name="imu_link"/>
+  <joint name="base_link_to_imu_joint" type="fixed">
+    <parent link="base_link"/>
+    <child link="imu_link"/>
+    <origin xyz="0.067 0 0.0145" rpy="0 0 0"/>
   </joint>
   <!-- Official OAK-D Pro description attached to the SolidWorks camera_base_link.

Commit message: localization stack hopefully final

File: src/bfmc_car_description/urdf/bfmc_car_description.urdf.xacro (robot description, xacro)
@@ -464,5 +464,5 @@
     <parent link="base_link"/>
     <child link="gps_tag_link"/>
-    <origin xyz="0.135 0 0.102" rpy="0 0 0"/>
+    <origin xyz="0.075 0 0.102" rpy="0 0 0"/>
   </joint>
   <!-- Rear IMU (BNO055) — position from SolidWorks assembly export -->
@@ -471,5 +471,5 @@
     <parent link="base_link"/>
     <child link="imu_link"/>
-    <origin xyz="0.067 0 0.0145" rpy="0 0 0"/>
+    <origin xyz="0.11 0 0.0145" rpy="0 0 0"/>
   </joint>
   <!-- Official OAK-D Pro description attached to the SolidWorks camera_base_link.
